File: Main Board/Xterminator 2.kicad_pcb (KiCad board)
At the start: 2 copper layers, 108.1 x 68 mm, 29 parts, among them SW1 SW_DP3T, U1 74LS10, U2 GAL16V8, U3 HM62256BLP

Commit message: Add files via upload
Connections:
- net /O12 renamed //Famicom.GND
Routing:
- net /GND: track 303.8 -> 306.9 mm
- net /A13: track 119.8 -> 120.8 mm
- net /Read.Top: track 66.2 -> 67.2 mm
- net /D1: track 100.8 -> 101.6 mm
- net /D0: track 121.0 -> 121.8 mm
- net /CIC.Out.P2.Top: track 63.7 -> 63.1 mm
