File: Main Board/Xterminator 2.kicad_sch (KiCad schematic)
At the start: 29 parts, among them SW1 SW_DP3T, U1 74LS10, U2 GAL16V8, U3 HM62256BLP

Commit message: Add files via upload
Connections:
- net A10.or.A11 renamed A10.and.A11
- net A3.or.A5.or.A6 renamed A3.and.A5.and.A6
- net A7.or.A8.or.A9 renamed A7.and.A8.and.A9
Changed lines of the file:
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@@
     (effects (font (size 1.27 1.27)) (justify right bottom))
   )
-  (label "A3.or.A5.or.A6" (at 234.95 92.71 180) (fields_autoplaced)
+  (label "A3.and.A5.and.A6" (at 234.95 92.71 180) (fields_autoplaced)
     (effects (font (size 1.27 1.27)) (justify right bottom))
   )
@@
     (effects (font (size 1.27 1.27)) (justify right bottom))
   )
-  (label "A3.or.A5.or.A6" (at 237.49 143.51 0) (fields_autoplaced)
+  (label "A3.and.A5.and.A6" (at 237.49 143.51 0) (fields_autoplaced)
     (effects (font (size 1.27 1.27)) (justify left bottom))
   )
@@
     (effects (font (size 1.27 1.27)) (justify left bottom))
   )
-  (label "A10.or.A11" (at 234.95 82.55 180) (fields_autoplaced)
+  (label "A10.and.A11" (at 234.95 82.55 180) (fields_autoplaced)
     (effects (font (size 1.27 1.27)) (justify right bottom))
   )
@@
     (effects (font (size 1.27 1.27)) (justify right bottom))
   )
-  (label "A7.or.A8.or.A9" (at 267.97 123.19 0) (fields_autoplaced)
+  (label "A7.and.A8.and.A9" (at 267.97 123.19 0) (fields_autoplaced)
     (effects (font (size 1.27 1.27)) (justify left bottom))
   )
@@
     (effects (font (size 1.27 1.27)) (justify left bottom))
   )
-  (label "A10.or.A11" (at 237.49 123.19 0) (fields_autoplaced)
+  (label "A10.and.A11" (at 237.49 123.19 0) (fields_autoplaced)
     (effects (font (size 1.27 1.27)) (justify left bottom))
   )
@@
     (effects (font (size 1.27 1.27)) (justify right bottom))
   )
-  (label "A7.or.A8.or.A9" (at 234.95 90.17 180) (fields_autoplaced)
-    (effects (font (size 1.27 1.27)) (justify right bottom))
-  )
+  (label "A7.and.A8.and.A9" (at 234.95 90.17 180) (fields_autoplaced)
+    (effects (font (size 1.27 1.27)) (justify right bottom))
+  )

Commit message: Add files via upload
Connections:
- net A0.Internal is gone; now on net A0: U3.10 (A0), U4.5 (Input), U5.10 (A0)
Changed lines of the file:
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@@
-    (effects (font (size 1.27 1.27)) (justify right bottom))
-  )
-  (label "A0.Internal" (at 24.13 147.32 180) (fields_autoplaced)
     (effects (font (size 1.27 1.27)) (justify right bottom))
   )
@@
     (effects (font (size 1.27 1.27)) (justify left bottom))
   )
+  (label "A0" (at 130.81 165.1 180) (fields_autoplaced)
+    (effects (font (size 1.27 1.27)) (justify right bottom))
+  )
   (label "Read.Bottom" (at 49.53 175.26 0) (fields_autoplaced)
     (effects (font (size 1.27 1.27)) (justify left bottom))
@@
     (effects (font (size 1.27 1.27)) (justify right bottom))
   )
+  (label "A0" (at 76.2 171.45 180) (fields_autoplaced)
+    (effects (font (size 1.27 1.27)) (justify right bottom))
+  )
   (label "A4" (at 85.09 67.31 180) (fields_autoplaced)
     (effects (font (size 1.27 1.27)) (justify right bottom))
@@
     (effects (font (size 1.27 1.27)) (justify right bottom))
   )
+  (label "A0" (at 24.13 147.32 180) (fields_autoplaced)
+    (effects (font (size 1.27 1.27)) (justify right bottom))
+  )
   (label "VCC" (at 85.09 102.87 180) (fields_autoplaced)
     (effects (font (size 1.27 1.27)) (justify right bottom))
@@
     (effects (font (size 1.27 1.27)) (justify right bottom))
   )
-  (label "A0.Internal" (at 130.81 165.1 180) (fields_autoplaced)
-    (effects (font (size 1.27 1.27)) (justify right bottom))
-  )
   (label "Reset" (at 24.13 101.6 180) (fields_autoplaced)
     (effects (font (size 1.27 1.27)) (justify right bottom))
@@
     (effects (font (size 1.27 1.27)) (justify left bottom))
   )
-  (label "A0.Internal" (at 76.2 171.45 180) (fields_autoplaced)
-    (effects (font (size 1.27 1.27)) (justify right bottom))
-  )
   (label "VCC" (at 24.13 104.14 180) (fields_autoplaced)

Commit message: Add files via upload
Connections:
- net O12 renamed /Famicom.GND
Changed lines of the file:
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@@
     (effects (font (size 1.27 1.27)) (justify right bottom))
   )
-  (label "O12" (at 231.14 54.61 180) (fields_autoplaced)
+  (label "{slash}Famicom.GND" (at 231.14 54.61 180) (fields_autoplaced)
     (effects (font (size 1.27 1.27)) (justify right bottom))
   )
@@
     (effects (font (size 1.27 1.27)) (justify left bottom))
   )
-  (label "O12" (at 231.14 52.07 180) (fields_autoplaced)
+  (label "{slash}Famicom.GND" (at 231.14 52.07 180) (fields_autoplaced)
     (effects (font (size 1.27 1.27)) (justify right bottom))
   )
@@
     (effects (font (size 1.27 1.27)) (justify left bottom))
   )
-  (label "O12" (at 260.35 95.25 0) (fields_autoplaced)
-    (effects (font (size 1.27 1.27)) (justify left bottom))
-  )
+  (label "{slash}Famicom.GND" (at 260.35 95.25 0) (fields_autoplaced)
+    (effects (font (size 1.27 1.27)) (justify left bottom))
+  )
